File: COMMS_circuit/PP_radio.kicad_sch (KiCad schematic)
At the start: 60 parts, among them J1 SMA, J2 SMA, U1 max19713etn+, U2 LTC5599IUF-PBF, U3 LTC5584IUF-PBF, U6 NSVG3117SG6T1G, U7 NSVG3117SG6T1G, U8 MAX2754EUA+

Commit message: Stick a RP2040 on the side and see if we can program an FPGA with it
Changed lines of the file:
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@@
 (kicad_sch
-	(version 20231120)
+	(version 20250114)
 	(generator "eeschema")
-	(generator_version "8.0")
+	(generator_version "9.0")
 	(paper "A4")
+	(text "Bandpass filters to\nAC couple and remove\nhigher order harmonics"
+		(exclude_from_sim no)
+		(at 152.146 34.036 0)
+		(effects
+			(font
+				(size 1 1)
+				(color 255 0 0 1)
+			)
+		)
+	)
+	(text "Demodulator"
+		(exclude_from_sim no)
+		(at 36.83 194.564 0)
+		(effects
+			(font
+				(size 5 5)
+				(thickness 1)
+				(bold yes)
+			)
+		)
+	)
+	(text "Modulator"
+		(exclude_from_sim no)
+		(at 146.558 73.406 0)
+		(effects
+			(font
+				(size 5 5)
+				(thickness 1)
+				(bold yes)
+			)
+		)
+	)
+	(text "Carrier LO"
+		(exclude_from_sim no)
+		(at 190.246 161.29 0)
+		(effects
+			(font
+				(size 5 5)
+				(thickness 1)
+				(bold yes)
+			)
+		)
+	)
+	(text "Analog Front End"
+		(exclude_from_sim no)
+		(at 46.736 109.728 0)
+		(effects
+			(font
+				(size 5 5)
+				(thickness 1)
+				(bold yes)
+			)
+		)
+	)
+	(text "Enabling DC offset correction so I\nhave the option to correct for it\nif I need to. God I hope I don't"
+		(exclude_from_sim no)
+		(at 72.644 182.626 0)
+		(effects
+			(font
+				(size 1 1)
+				(color 255 0 0 1)
+			)
+		)
+	)
+	(text "Low pass filter\nmaybe VGA as\n well"
+		(exclude_from_sim no)
+		(at 111.506 131.572 0)
+		(effects
+			(font
+				(size 1 1)
+				(color 255 0 0 1)
+			)
+		)
+	)
+	(text "Amplifiers"
+		(exclude_from_sim no)
+		(at 145.288 110.49 0)
+		(effects
+			(font
+				(size 5 5)
+				(thickness 1)
+				(bold yes)
+			)
+		)
+	)
+	(text "Depends on \ncontroller\nlogic level"
+		(exclude_from_sim no)
+		(at 18.796 69.85 0)
+		(effects
+			(font
+				(size 1 1)
+				(color 255 0 0 1)
+			)
+		)
+	)
 	(junction
 		(at 148.59 96.52)
@@
 		)
 	)
-	(text "Bandpass filters to\nAC couple and remove\nhigher order harmonics"
-		(exclude_from_sim no)
-		(at 152.146 34.036 0)
-		(effects
-			(font
-				(size 1 1)
-				(color 255 0 0 1)
-			)
-		)
-	)
-	(text "Demodulator"
-		(exclude_from_sim no)
-		(at 36.83 194.564 0)
-		(effects
-			(font
-				(size 5 5)
-				(thickness 1)
-				(bold yes)
-			)
-		)
-	)
-	(text "Modulator"
-		(exclude_from_sim no)
-		(at 146.558 73.406 0)
-		(effects
-			(font
-				(size 5 5)
-				(thickness 1)
-				(bold yes)
-			)
-		)
-	)
-	(text "Carrier LO"
-		(exclude_from_sim no)
-		(at 190.246 161.29 0)
-		(effects
-			(font
-				(size 5 5)
-				(thickness 1)
-				(bold yes)
-			)
-		)
-	)
-	(text "Analog Front End"
-		(exclude_from_sim no)
-		(at 46.736 109.728 0)
-		(effects
-			(font
-				(size 5 5)
-				(thickness 1)
-				(bold yes)
-			)
-		)
-	)
-	(text "Enabling DC offset correction so I\nhave the option to correct for it\nif I need to. God I hope I don't"
-		(exclude_from_sim no)
-		(at 72.644 182.626 0)
-		(effects
-			(font
-				(size 1 1)
-				(color 255 0 0 1)
-			)
-		)
-	)
-	(text "Low pass filter\nmaybe VGA as\n well"
-		(exclude_from_sim no)
-		(at 111.506 131.572 0)
-		(effects
-			(font
-				(size 1 1)
-				(color 255 0 0 1)
-			)
-		)
-	)
-	(text "Amplifiers"
-		(exclude_from_sim no)
-		(at 145.288 110.49 0)
-		(effects
-			(font
-				(size 5 5)
-				(thickness 1)
-				(bold yes)
-			)
-		)
-	)
-	(text "Depends on \ncontroller\nlogic level"
-		(exclude_from_sim no)
-		(at 18.796 69.85 0)
-		(effects
-			(font
-				(size 1 1)
-				(color 255 0 0 1)
-			)
-		)
-	)
 	(label "RX_RF"
 		(at 21.59 148.59 180)
@@
 		(at 152.4 62.23)
 		(size 12.7 4.826)
+		(exclude_from_sim no)
+		(in_bom yes)
+		(on_board yes)
+		(dnp no)
 		(stroke
 			(width 0.1524)
@@
 		(at 124.46 142.24)
 		(size 12.7 4.826)
+		(exclude_from_sim no)
+		(in_bom yes)
+		(on_board yes)
+		(dnp no)
 		(stroke
 			(width 0.1524)
@@
 		(at 152.4 39.37)
 		(size 12.7 4.826)
+		(exclude_from_sim no)
+		(in_bom yes)
+		(on_board yes)
+		(dnp no)
 		(stroke
 			(width 0.1524)
@@
 		(at 124.46 149.86)
 		(size 12.7 4.826)
+		(exclude_from_sim no)
+		(in_bom yes)
+		(on_board yes)
+		(dnp no)
 		(stroke
 			(width 0.1524)
@@
 		(at 124.46 134.62)
 		(size 12.7 4.826)
+		(exclude_from_sim no)
+		(in_bom yes)
+		(on_board yes)
+		(dnp no)
 		(stroke
 			(width 0.1524)
@@
 		(at 124.46 127)
 		(size 12.7 4.826)
+		(exclude_from_sim no)
+		(in_bom yes)
+		(on_board yes)
+		(dnp no)
 		(stroke
 			(width 0.1524)
@@
 		(at 152.4 54.61)
 		(size 12.7 4.826)
+		(exclude_from_sim no)
+		(in_bom yes)
+		(on_board yes)
+		(dnp no)
 		(stroke
 			(width 0.1524)
@@
 		(at 152.4 46.99)
 		(size 12.7 4.826)
+		(exclude_from_sim no)
+		(in_bom yes)
+		(on_board yes)
+		(dnp no)
 		(stroke
 			(width 0.1524)
