File: COMMS_circuit/Power.kicad_sch (KiCad schematic)
At the start: 53 parts, among them J4 Conn_01x02_Pin, U12 ADP7105ACPZ-R7, U13 ADP7105ACPZ-R7, U14 TPS2121RUXR, U4 ADP7105ACPZ-3.3-R7, U5 ADP7105ACPZ-5.0-R7

Commit message: Changes I missed cause id been staring at it to long
Other:
- moved on the sheet: C100, C101, C60, C61, C62, C63, C85, C86, C87, C88, C89, C90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
