File: COMMS_circuit/RX_Filter.kicad_sch (KiCad schematic)
At the start: 5 parts

Commit message: testing opsec update
Parts:
- L16: renamed from L19; value 12u -> 360n
Changed lines of the file:
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@@
 		(shape output)
 		(at 78.74 81.28 0)
-		(fields_autoplaced yes)
 		(effects
 			(font
@@
 		(shape input)
 		(at 64.77 81.28 180)
-		(fields_autoplaced yes)
 		(effects
 			(font
@@
 					(unit 1)
 				)
+				(path "/bdd480c2-e959-4f78-bdcb-24d46c5e40e4/ede84ad4-bf81-4ce0-9af5-65c60d47287f/277dc9e8-b560-4155-8275-da18d2dcac37"
+					(reference "C47")
+					(unit 1)
+				)
 				(path "/bdd480c2-e959-4f78-bdcb-24d46c5e40e4/ede84ad4-bf81-4ce0-9af5-65c60d47287f/65289467-89f5-4c62-a2e7-aed485fdf276"
 					(reference "C45")
@@
 					(unit 1)
 				)
-				(path "/bdd480c2-e959-4f78-bdcb-24d46c5e40e4/ede84ad4-bf81-4ce0-9af5-65c60d47287f/277dc9e8-b560-4155-8275-da18d2dcac37"
-					(reference "C47")
-					(unit 1)
-				)
 			)
 		)
@@
 					(unit 1)
 				)
+				(path "/bdd480c2-e959-4f78-bdcb-24d46c5e40e4/ede84ad4-bf81-4ce0-9af5-65c60d47287f/277dc9e8-b560-4155-8275-da18d2dcac37"
+					(reference "R13")
+					(unit 1)
+				)
 				(path "/bdd480c2-e959-4f78-bdcb-24d46c5e40e4/ede84ad4-bf81-4ce0-9af5-65c60d47287f/65289467-89f5-4c62-a2e7-aed485fdf276"
 					(reference "R15")
@@
 					(unit 1)
 				)
-				(path "/bdd480c2-e959-4f78-bdcb-24d46c5e40e4/ede84ad4-bf81-4ce0-9af5-65c60d47287f/277dc9e8-b560-4155-8275-da18d2dcac37"
-					(reference "R13")
-					(unit 1)
-				)
 			)
 		)
@@
 					(unit 1)
 				)
+				(path "/bdd480c2-e959-4f78-bdcb-24d46c5e40e4/ede84ad4-bf81-4ce0-9af5-65c60d47287f/277dc9e8-b560-4155-8275-da18d2dcac37"
+					(reference "C43")
+					(unit 1)
+				)
 				(path "/bdd480c2-e959-4f78-bdcb-24d46c5e40e4/ede84ad4-bf81-4ce0-9af5-65c60d47287f/65289467-89f5-4c62-a2e7-aed485fdf276"
 					(reference "C41")
@@
 					(unit 1)
 				)
-				(path "/bdd480c2-e959-4f78-bdcb-24d46c5e40e4/ede84ad4-bf81-4ce0-9af5-65c60d47287f/277dc9e8-b560-4155-8275-da18d2dcac37"
-					(reference "C43")
-					(unit 1)
-				)
 			)
 		)
@@
 		(dnp no)
 		(fields_autoplaced yes)
-		(property "Reference" "L19"
+		(property "Reference" "L16"
 			(at 71.12 76.2 90)
 			(effects
@@
 			)
 		)
-		(property "Value" "12u"
+		(property "Value" "360n"
 			(at 71.12 78.74 90)
 			(effects
@@
 		(instances
 			(project "COMMS_circuit"
+				(path "/bdd480c2-e959-4f78-bdcb-24d46c5e40e4/ede84ad4-bf81-4ce0-9af5-65c60d47287f/060a43dc-e3c7-438b-87dd-8d33e58dd6d2"
+					(reference "L16")
+					(unit 1)
+				)
 				(path "/bdd480c2-e959-4f78-bdcb-24d46c5e40e4/ede84ad4-bf81-4ce0-9af5-65c60d47287f/277dc9e8-b560-4155-8275-da18d2dcac37"
 					(reference "L19")
-					(unit 1)
-				)
-				(path "/bdd480c2-e959-4f78-bdcb-24d46c5e40e4/ede84ad4-bf81-4ce0-9af5-65c60d47287f/060a43dc-e3c7-438b-87dd-8d33e58dd6d2"
-					(reference "L16")
 					(unit 1)
 				)
@@
 					(unit 1)
 				)
+				(path "/bdd480c2-e959-4f78-bdcb-24d46c5e40e4/ede84ad4-bf81-4ce0-9af5-65c60d47287f/277dc9e8-b560-4155-8275-da18d2dcac37"
+					(reference "#PWR031")
+					(unit 1)
+				)
 				(path "/bdd480c2-e959-4f78-bdcb-24d46c5e40e4/ede84ad4-bf81-4ce0-9af5-65c60d47287f/65289467-89f5-4c62-a2e7-aed485fdf276"
 					(reference "#PWR034")
@@
 					(unit 1)
 				)
-				(path "/bdd480c2-e959-4f78-bdcb-24d46c5e40e4/ede84ad4-bf81-4ce0-9af5-65c60d47287f/277dc9e8-b560-4155-8275-da18d2dcac37"
-					(reference "#PWR031")
-					(unit 1)
-				)
 			)
 		)
@@
 					(unit 1)
 				)
+				(path "/bdd480c2-e959-4f78-bdcb-24d46c5e40e4/ede84ad4-bf81-4ce0-9af5-65c60d47287f/277dc9e8-b560-4155-8275-da18d2dcac37"
+					(reference "C36")
+					(unit 1)
+				)
 				(path "/bdd480c2-e959-4f78-bdcb-24d46c5e40e4/ede84ad4-bf81-4ce0-9af5-65c60d47287f/65289467-89f5-4c62-a2e7-aed485fdf276"
 					(reference "C38")
@@
 					(unit 1)
 				)
-				(path "/bdd480c2-e959-4f78-bdcb-24d46c5e40e4/ede84ad4-bf81-4ce0-9af5-65c60d47287f/277dc9e8-b560-4155-8275-da18d2dcac37"
-					(reference "C36")
-					(unit 1)
-				)
 			)
 		)
@@
 		(dnp no)
 		(fields_autoplaced yes)
-		(property "Reference" "#PWR0101"
+		(property "Reference" "#PWR033"
 			(at 87.63 99.06 0)
 			(effects
@@
 		(instances
 			(project "COMMS_circuit"
+				(path "/bdd480c2-e959-4f78-bdcb-24d46c5e40e4/ede84ad4-bf81-4ce0-9af5-65c60d47287f/060a43dc-e3c7-438b-87dd-8d33e58dd6d2"
+					(reference "#PWR033")
+					(unit 1)
+				)
 				(path "/bdd480c2-e959-4f78-bdcb-24d46c5e40e4/ede84ad4-bf81-4ce0-9af5-65c60d47287f/277dc9e8-b560-4155-8275-da18d2dcac37"
 					(reference "#PWR0101")
 					(unit 1)
 				)
-				(path "/bdd480c2-e959-4f78-bdcb-24d46c5e40e4/ede84ad4-bf81-4ce0-9af5-65c60d47287f/060a43dc-e3c7-438b-87dd-8d33e58dd6d2"
-					(reference "#PWR033")
-					(unit 1)
-				)

Commit message: Stick a RP2040 on the side and see if we can program an FPGA with it
Changed lines of the file:
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@@
 (kicad_sch
-	(version 20231120)
+	(version 20250114)
 	(generator "eeschema")
-	(generator_version "8.0")
+	(generator_version "9.0")
 	(paper "A")
 	(junction
